File: Controller/Controller.kicad_pcb (KiCad board)
At the start: 2 copper layers, 132 x 132 mm, 24 parts, among them J1 USB_B, SW2 SW_Push, SW3 SW_Push, SW4 SW_Push, SW5 SW_Push, SW6 SW_Push, SW7 SW_Push, SW8 SW_Push, SW9 SW_Push

Commit message: Fix mistakes
Parts:
- J1, R2: moved to F.Cu
- LDR_R1: footprint Resistor_THT:R_Axial_DIN0204_L3.6mm_D1.6mm_P5.08mm_Horizontal -> Resistor_THT:R_Axial_DIN0204_L3.6mm_D1.6mm_P7.62mm_Horizontal; moved to F.Cu
- MOUNTING_HOLE_1: renamed from HOLE_1; value MountingHole_8.4mm_M8 -> M8_8.4mm; footprint MountingHole:MountingHole_8.4mm_M8 -> MountingHole:MountingHole_8.4mm_M8_ETIMC
- MOUNTING_HOLE_2: renamed from HOLE_2; value MountingHole_8.4mm_M8 -> M8_8.4mm; footprint MountingHole:MountingHole_8.4mm_M8 -> MountingHole:MountingHole_8.4mm_M8_ETIMC
- MOUNTING_HOLE_3: renamed from HOLE_3; value MountingHole_8.4mm_M8 -> M8_8.4mm; footprint MountingHole:MountingHole_8.4mm_M8 -> MountingHole:MountingHole_8.4mm_M8_ETIMC
- MOUNTING_HOLE_4: renamed from HOLE_4; value MountingHole_8.4mm_M8 -> M8_8.4mm; footprint MountingHole:MountingHole_8.4mm_M8 -> MountingHole:MountingHole_8.4mm_M8_ETIMC
- NFC-1: footprint Connector_PinHeader_2.54mm:PinHeader_1x07_P2.54mm_Vertical -> Connector_PinHeader_2.54mm:PinHeader_1x08_P2.54mm_Vertical; moved to F.Cu
- POT_1: renamed from RV4; footprint Potentiometer_THT:Potentiometer_Vishay_148-149_Single_Vertical -> Potentiometer_THT:Potentiometer_Vishay_148-149_Single_Vertical_ETIMC
- POT_1: renamed from RV1; footprint Potentiometer_THT:Potentiometer_Vishay_148-149_Single_Vertical -> Potentiometer_THT:Potentiometer_Vishay_148-149_Single_Vertical_ETIMC
- POT_2: renamed from RV3; footprint Potentiometer_THT:Potentiometer_Vishay_148-149_Single_Vertical -> Potentiometer_THT:Potentiometer_Vishay_148-149_Single_Vertical_ETIMC
- POT_3: renamed from RV2; footprint Potentiometer_THT:Potentiometer_Vishay_148-149_Single_Vertical -> Potentiometer_THT:Potentiometer_Vishay_148-149_Single_Vertical_ETIMC
- moved ON/OFF-Switch1 5.18 mm to (125.2, 24.5), turned to -90 degrees
- moved LDR_R1 0.20 mm to (121.0, 33.9)
- moved R2 0.11 mm to (128.0, 35.0), turned to 90 degrees
- turned J1 to 180 degrees
- turned NFC-1 to 90 degrees
- renumbered SW2 to SWITCH_1, SW4 to SWITCH_2, SW6 to SWITCH_3, SW8 to SWITCH_4, SW3 to SWITCH_5, SW5 to SWITCH_6, SW7 to SWITCH_7, SW9 to SWITCH_8
Routing:
- net Net-(NFC-1-SS/SDA/RX): track 0.00 -> 23.3 mm
- net Net-(Multiplexer1-A0): track 81.4 -> 88.9 mm
- net Net-(Multiplexer1-S0): track 42.4 -> 49.2 mm
- net Net-(Multiplexer1-S1): track 44.4 -> 49.7 mm
- net Net-(Multiplexer1-S2): track 63.0 -> 60.8 mm
- net Net-(Multiplexer1-A4): track 64.8 -> 63.4 mm
- net Net-(J1-VBUS): track 20.5 -> 19.7 mm
- net GND: track 640.1 -> 639.5 mm
Other:
- board text added: "ETIMC Controller v3 De Danske Geder SpilTek 2022"
- board text removed: "ETIMC Controller v1 De Danske Geder SpilTek 2022"
