File: Controller/Controller.kicad_pcb (KiCad board)
At the start: 2 copper layers, 132 x 132 mm, 24 parts, among them J1 USB_B

Commit message: Update schematic and schematic PDF
Parts:
- removed LDR_R1: ???, Resistor_THT:R_Axial_DIN0204_L3.6mm_D1.6mm_P7.62mm_Horizontal
- removed R2: LDR03, Connector_PinHeader_2.54mm:PinHeader_1x02_P2.54mm_Vertical
- added LDR1: LDR03, Connector_PinHeader_2.54mm:PinHeader_1x02_P2.54mm_Vertical, B.Cu at (128.0, 35.0)
- added LDR1_LED1: RED, Connector_PinHeader_2.54mm:PinHeader_1x02_P2.54mm_Vertical, B.Cu at (144.5, 104.0)
- added LDR1_R1: ???, Resistor_THT:R_Axial_DIN0204_L3.6mm_D1.6mm_P7.62mm_Horizontal, B.Cu at (121.0, 33.9)
- added LED1_R1: 120, Resistor_THT:R_Axial_DIN0204_L3.6mm_D1.6mm_P7.62mm_Horizontal, B.Cu at (144.5, 114.0)
- NFC-1: moved to B.Cu
- POT_1: footprint Potentiometer_THT:Potentiometer_Vishay_148-149_Single_Vertical_ETIMC -> Potentiometer_THT:Potentiometer_Vishay_148-149_Single_Vertical
- POT_2: renamed from POT_3; footprint Potentiometer_THT:Potentiometer_Vishay_148-149_Single_Vertical_ETIMC -> Potentiometer_THT:Potentiometer_Vishay_148-149_Single_Vertical
- POT_3: renamed from POT_2; footprint Potentiometer_THT:Potentiometer_Vishay_148-149_Single_Vertical_ETIMC -> Potentiometer_THT:Potentiometer_Vishay_148-149_Single_Vertical
- POT_4: renamed from POT_1; footprint Potentiometer_THT:Potentiometer_Vishay_148-149_Single_Vertical_ETIMC -> Potentiometer_THT:Potentiometer_Vishay_148-149_Single_Vertical
- USB_B1: renamed from J1; moved to B.Cu
- turned NFC-1 to -90 degrees
- turned USB_B1 to 0 degrees
Connections:
- SWITCH_1 pad 2: Net-(SW2-Pad2) -> GND
- SWITCH_2 pad 2: Net-(SW2-Pad2) -> GND
- SWITCH_3 pad 2: Net-(SW2-Pad2) -> GND
- SWITCH_4 pad 2: Net-(SW2-Pad2) -> GND
- SWITCH_5 pad 2: Net-(SW2-Pad2) -> GND
- SWITCH_6 pad 2: Net-(SW2-Pad2) -> GND
- SWITCH_7 pad 2: Net-(SW2-Pad2) -> GND
- SWITCH_8 pad 2: Net-(SW2-Pad2) -> GND
Routing:
- net GND: track 639.5 -> 899.0 mm
- net Net-(SW2-Pad2): track 214.4 -> 0.00 mm
- net 3V3: track 489.9 -> 550.6 mm
- net Net-(LDR1_LED1-A): track 0.00 -> 7.50 mm
Other:
- board text added: "ETIMC Controller v6 De Danske Geder SpilTek 2022"
- board text removed: "ETIMC Controller v3 De Danske Geder SpilTek 2022"
