File: Controller/Controller.kicad_sch (KiCad schematic)
At the start: 33 parts, among them J1 USB_B, SW2 SW_Push, SW3 SW_Push, SW4 SW_Push, SW5 SW_Push, SW6 SW_Push, SW7 SW_Push, SW8 SW_Push, SW9 SW_Push

Commit message: Fix i2c
Connections:
- net at SW9.1: now also PICO-1.32 (I2C1_SCL/ADC1/GP27); no longer PICO-1.26 (I2C0_SDA/GP20)
- net GP27 renamed GP20
- net GP20: now also PICO-1.26 (I2C0_SDA/GP20); no longer PICO-1.32 (I2C1_SCL/ADC1/GP27)

Commit message: Fix mistakes
Parts:
- NFC-1: footprint Connector_PinHeader_2.54mm:PinHeader_1x07_P2.54mm_Vertical -> Connector_PinHeader_2.54mm:PinHeader_1x08_P2.54mm_Vertical
Changed lines of the file:
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@@
 			)
 		)
-		(property "Footprint" "Connector_PinHeader_2.54mm:PinHeader_1x07_P2.54mm_Vertical"
+		(property "Footprint" "Connector_PinHeader_2.54mm:PinHeader_1x08_P2.54mm_Vertical"
 			(at 38.1 76.2 0)
 			(effects

Commit message: Update schematic and schematic PDF
Parts:
- added LDR1_LED1: RED, Connector_PinHeader_2.54mm:PinHeader_1x02_P2.54mm_Vertical, symbol Device:LED
- added LED1_R1: 120, Resistor_THT:R_Axial_DIN0204_L3.6mm_D1.6mm_P7.62mm_Horizontal, symbol Device:R
- LDR1_R1: renamed from LDR_R1; footprint Resistor_THT:R_Axial_DIN0204_L3.6mm_D1.6mm_P5.08mm_Horizontal -> Resistor_THT:R_Axial_DIN0204_L3.6mm_D1.6mm_P7.62mm_Horizontal
- renumbered R2 to LDR1, RV1 to POT_1, RV2 to POT_2, RV3 to POT_3, RV4 to POT_4, R1 to R_LED1, SW2 to SWITCH_1, SW3 to SWITCH_2, SW4 to SWITCH_3, SW5 to SWITCH_4, SW9 to SWITCH_5, SW8 to SWITCH_6, SW7 to SWITCH_7, SW6 to SWITCH_8, J1 to USB_B1
Connections:
- net 3V3: now also LED1_R1.2
- net GND: now also SWITCH_1.2, SWITCH_2.2, SWITCH_3.2, SWITCH_4.2, SWITCH_5.2, SWITCH_6.2, SWITCH_7.2, SWITCH_8.2, LDR1_LED1.1 (K)
- net at PICO-1.19 (I2C1_SDA/SPI1_SCK/GP14): now also SWITCH_5.1; no longer SWITCH_2.1
- net at PICO-1.20 (I2C1_SCL/SPI1_TX/GP15): now also SWITCH_2.1; no longer SWITCH_3.1
- net at PICO-1.21 (UART0_TX/I2C0_SDA/SPI0_RX/GP16): now also SWITCH_6.1; no longer SWITCH_4.1
- net at PICO-1.22 (UART0_RX/I2C0_SCL/SPI0_CSN/GP17): now also SWITCH_3.1; no longer SWITCH_8.1
- net at PICO-1.25 (I2C1_SCL/SPI0_TX/GP19): now also SWITCH_4.1; no longer SWITCH_6.1
- net at PICO-1.32 (I2C1_SCL/ADC1/GP27): now also SWITCH_8.1; no longer SWITCH_5.1
- new net: LDR1_LED1.2 (A), LED1_R1.1
